Commit message: Gravity fix

File: src/trr_robot_desc/robots/trr_robot.urdf.xacro (robot description, xacro)
@@ -13,9 +13,9 @@
     <xacro:property name="wheel_xoff" value="0.215"/>
     <!-- =============== Link & Joint =============== -->
-    <link name="world"></link>
+    <link name="base_footprint"></link>
     <joint name="base_joint" type="fixed">
-        <parent link="world"/>
+        <parent link="base_footprint"/>
         <child link="base_link"/>
-        <origin xyz="0.0 0.0 ${-(wheel_radius+wheel_zoff)}" rpy="0 0 0"/>
+        <origin xyz="0.0 0.0 0.075" rpy="0 0 0"/>
     </joint>
     <link name="base_link">
@@ -52,4 +52,10 @@
                 </material>
             </visual>
+            <collision>
+                <origin xyz="0 0 0" rpy="${pi/2} 0 0"/>
+                <geometry>
+                    <cylinder radius="${wheel_radius}" length="${wheel_width}"/>
+                </geometry>
+            </collision>
             <inertial>
                 <origin xyz="0 0 0"/>

Commit message: Simulated robot can be controlled with game controller!

File: src/trr_robot_desc/robots/trr_robot.urdf.xacro (robot description, xacro)
@@ -71,8 +71,8 @@
         </joint>
     </xacro:macro>
-    <xacro:wheel prefix="drivewhl_1" x_reflect="-1" y_reflect="1" />
-    <xacro:wheel prefix="drivewhl_2" x_reflect="-1" y_reflect="-1" />
-    <xacro:wheel prefix="drivewhl_3" x_reflect="1" y_reflect="1" />
-    <xacro:wheel prefix="drivewhl_4" x_reflect="1" y_reflect="-1" />
+    <xacro:wheel prefix="drivewhl_fl" x_reflect="1" y_reflect="1" />
+    <xacro:wheel prefix="drivewhl_fr" x_reflect="1" y_reflect="-1" />
+    <xacro:wheel prefix="drivewhl_rl" x_reflect="-1" y_reflect="1" />
+    <xacro:wheel prefix="drivewhl_rr" x_reflect="-1" y_reflect="-1" />
     <!-- =============== Gazebo =============== -->
     <xacro:macro name="base_gazebo_v0">
@@ -91,8 +91,8 @@
     </xacro:macro>
     <xacro:base_gazebo_v0/>
-    <xacro:wheel_gazebo_v0 prefix="drivewhl_1"/>
-    <xacro:wheel_gazebo_v0 prefix="drivewhl_2"/>
-    <xacro:wheel_gazebo_v0 prefix="drivewhl_3"/>
-    <xacro:wheel_gazebo_v0 prefix="drivewhl_4"/>
+    <xacro:wheel_gazebo_v0 prefix="drivewhl_fl"/>
+    <xacro:wheel_gazebo_v0 prefix="drivewhl_fr"/>
+    <xacro:wheel_gazebo_v0 prefix="drivewhl_rl"/>
+    <xacro:wheel_gazebo_v0 prefix="drivewhl_rr"/>
     <xacro:trr_robot_gazebo/>
     <xacro:trr_robot_ros2_control/>

File: src/trr_robot_desc/ros2_control/trr_robot.ros2_control.xacro (robot description, xacro)
@@ -6,8 +6,8 @@
           <plugin>gz_ros2_control/GazeboSimSystem</plugin>
       </hardware>
-      <joint name="drivewhl_1_joint">
+      <joint name="drivewhl_fl_joint">
         <command_interface name="velocity">
-          <param name="min">-1</param>
-          <param name="max">1</param>
+          <param name="min">-7.5</param>
+          <param name="max">7.5</param>
         </command_interface>
         <state_interface name="position"/>
@@ -15,8 +15,8 @@
         <state_interface name="effort"/>
       </joint>
-      <joint name="drivewhl_2_joint">
+      <joint name="drivewhl_fr_joint">
         <command_interface name="velocity">
-          <param name="min">-1</param>
-          <param name="max">1</param>
+          <param name="min">-7.5</param>
+          <param name="max">7.5</param>
         </command_interface>
         <state_interface name="position"/>
@@ -24,8 +24,8 @@
         <state_interface name="effort"/>
       </joint>
-      <joint name="drivewhl_3_joint">
+      <joint name="drivewhl_rl_joint">
         <command_interface name="velocity">
-          <param name="min">-1</param>
-          <param name="max">1</param>
+          <param name="min">-7.5</param>
+          <param name="max">7.5</param>
         </command_interface>
         <state_interface name="position"/>
@@ -33,8 +33,8 @@
         <state_interface name="effort"/>
       </joint>
-      <joint name="drivewhl_4_joint">
+      <joint name="drivewhl_rr_joint">
         <command_interface name="velocity">
-          <param name="min">-1</param>
-          <param name="max">1</param>
+          <param name="min">-7.5</param>
+          <param name="max">7.5</param>
         </command_interface>
         <state_interface name="position"/>
