Commit message: Fixes to get it back up and running

File: src/trr_robot/description/depth_camera.xacro (robot description, xacro)
@@ -1,4 +1,9 @@
 <?xml version="1.0"?>
 <robot xmlns:xacro="http://www.ros.org/wiki/xacro" >
+    <gazebo>
+        <plugin filename="gz-sim-sensors-system" name="gz::sim::systems::Sensors">
+            <render_engine>ogre2</render_engine>
+        </plugin>
+    </gazebo>
     <joint name="camera_joint" type="fixed">
         <parent link="base_link"/>
@@ -26,17 +31,18 @@
             <always_on>true</always_on>
             <visualize>true</visualize>
-            <update_rate>30</update_rate>
+            <update_rate>10</update_rate>
             <topic>camera/image_raw</topic>
             <gz_frame_id>camera_rgb_frame</gz_frame_id>
             <camera>
                 <camera_info_topic>camera/camera_info</camera_info_topic>
-                <horizontal_fov>1.047</horizontal_fov>
+                <horizontal_fov>1.089</horizontal_fov>
                 <image>
-                    <width>320</width>
-                    <height>240</height>
+                    <format>B8G8R8</format>
+                    <width>640</width>
+                    <height>480</height>
                 </image>
                 <clip>
-                    <near>0.1</near>
-                    <far>100</far>
+                    <near>0.05</near>
+                    <far>8.0</far>
                 </clip>
             </camera>

File: src/trr_robot/description/robot_core.xacro (robot description, xacro)
@@ -1,5 +1,4 @@
 <?xml version="1.0"?>
 <robot xmlns:xacro="http://www.ros.org/wiki/xacro" name="trr_robot">
-    <xacro:include filename="$(find trr_robot_desc)/ros2_control/ros2_control.xacro" />
     <xacro:property name="base_width" value="0.4572"/>
     <xacro:property name="base_length" value="0.5588"/>
@@ -93,5 +92,4 @@
     <xacro:wheel_gazebo_v0 prefix="drivewhl_rl"/>
     <xacro:wheel_gazebo_v0 prefix="drivewhl_rr"/>
-    <xacro:trr_robot_gazebo/>
-    <xacro:trr_robot_ros2_control/>
+    <xacro:include filename="ros2_control.xacro" />
 </robot>

File: src/trr_robot/description/ros2_control.xacro (robot description, xacro)
@@ -1,51 +1,49 @@
 <?xml version="1.0"?>
 <robot xmlns:xacro="http://www.ros.org/wiki/xacro">
-  <xacro:macro name="trr_robot_ros2_control">
+    <gazebo>
+        <plugin filename="gz_ros2_control-system" name="gz_ros2_control::GazeboSimROS2ControlPlugin">
+            <parameters>$(find trr_robot)/config/controllers.yaml</parameters>
+        </plugin>
+    </gazebo>
     <ros2_control name="trr" type="system">
-      <hardware>
-          <plugin>gz_ros2_control/GazeboSimSystem</plugin>
-      </hardware>
-      <joint name="drivewhl_fl_joint">
-        <command_interface name="velocity">
-          <param name="min">-20</param>
-          <param name="max">20</param>
-        </command_interface>
-        <state_interface name="position"/>
-        <state_interface name="velocity"/>
-        <state_interface name="effort"/>
-      </joint>
-      <joint name="drivewhl_fr_joint">
-        <command_interface name="velocity">
-          <param name="min">-20</param>
-          <param name="max">20</param>
-        </command_interface>
-        <state_interface name="position"/>
-        <state_interface name="velocity"/>
-        <state_interface name="effort"/>
-      </joint>
-      <joint name="drivewhl_rl_joint">
-        <command_interface name="velocity">
-          <param name="min">-20</param>
-          <param name="max">20</param>
-        </command_interface>
-        <state_interface name="position"/>
-        <state_interface name="velocity"/>
-        <state_interface name="effort"/>
-      </joint>
-      <joint name="drivewhl_rr_joint">
-        <command_interface name="velocity">
-          <param name="min">-20</param>
-          <param name="max">20</param>
-        </command_interface>
-        <state_interface name="position"/>
-        <state_interface name="velocity"/>
-        <state_interface name="effort"/>
-      </joint>
+        <hardware>
+            <plugin>gz_ros2_control/GazeboSimSystem</plugin>
+        </hardware>
+        <joint name="drivewhl_fl_joint">
+            <command_interface name="velocity">
+                <param name="min">-20</param>
+                <param name="max">20</param>
+            </command_interface>
+            <state_interface name="position"/>
+            <state_interface name="velocity"/>
+            <state_interface name="effort"/>
+        </joint>
+        <joint name="drivewhl_fr_joint">
+            <command_interface name="velocity">
+                <param name="min">-20</param>
+                <param name="max">20</param>
+            </command_interface>
+            <state_interface name="position"/>
+            <state_interface name="velocity"/>
+            <state_interface name="effort"/>
+        </joint>
+        <joint name="drivewhl_rl_joint">
+            <command_interface name="velocity">
+                <param name="min">-20</param>
+                <param name="max">20</param>
+            </command_interface>
+            <state_interface name="position"/>
+            <state_interface name="velocity"/>
+            <state_interface name="effort"/>
+        </joint>
+        <joint name="drivewhl_rr_joint">
+            <command_interface name="velocity">
+                <param name="min">-20</param>
+                <param name="max">20</param>
+            </command_interface>
+            <state_interface name="position"/>
+            <state_interface name="velocity"/>
+            <state_interface name="effort"/>
+        </joint>
     </ros2_control>
-    <gazebo>
-      <plugin filename="gz_ros2_control-system" name="gz_ros2_control::GazeboSimROS2ControlPlugin">
-        <parameters>$(find trr_robot_desc)/config/trr_robot_sim.yaml</parameters>
-      </plugin>
-    </gazebo>
-  </xacro:macro>
 </robot>

File: src/trr_robot/description/trr_robot.urdf.xacro (robot description, xacro)
@@ -2,4 +2,4 @@
 <robot xmlns:xacro="http://www.ros.org/wiki/xacro" name="trr_robot">
     <xacro:include filename="robot_core.xacro"/>
-    <xacro:include filename="depth_camera.xacro" />
+    <xacro:include filename="depth_camera.xacro"/>
 </robot>
