Commit message: Switching to using differential drive gazebo plugin

File: src/trr_robot/description/gz.xacro (robot description, xacro)
@@ -7,4 +7,20 @@
         </plugin>
         <plugin filename="gz-sim-joint-state-publisher-system" name="gz::sim::systems::JointStatePublisher"></plugin>
+        <!-- Diff drive plugin -->
+        <plugin filename="gz-sim-diff-drive-system" name="gz::sim::systems::DiffDrive">
+            <num_wheel_pairs>2</num_wheel_pairs>
+            <left_joint>drivewhl_fl_joint</left_joint>
+            <left_joint>drivewhl_rl_joint</left_joint>
+            <right_joint>drivewhl_fr_joint</right_joint>
+            <right_joint>drivewhl_rr_joint</right_joint>
+            <wheel_separation>0.5</wheel_separation>
+            <wheel_radius>0.2</wheel_radius>
+            <odom_publish_frequency>30</odom_publish_frequency>
+            <topic>/cmd_vel</topic>
+            <odom_topic>odom</odom_topic>
+            <tf_topic>/tf</tf_topic>
+            <frame_id>odom</frame_id>
+            <child_frame_id>base_footprint</child_frame_id>
+        </plugin>
     </gazebo>
     <!-- ............................. ground truth .................................... -->
@@ -41,3 +57,23 @@
         </sensor>
     </gazebo>
+    <!-- ........................... Wheels and Base and Stuff ................................... -->
+    <xacro:macro name="base_gazebo_v0">
+        <gazebo reference="base_link">
+            <selfCollide>false</selfCollide>
+            <mu1 value="0.05" />
+            <mu2 value="0.05" />
+        </gazebo>
+    </xacro:macro>
+    <xacro:macro name="wheel_gazebo_v0" params="prefix">
+        <gazebo reference="${prefix}_link">
+            <selfCollide>false</selfCollide>
+            <mu1 value="1.2" />
+            <mu2 value="1.2" />
+        </gazebo>
+    </xacro:macro>
+    <xacro:base_gazebo_v0/>
+    <xacro:wheel_gazebo_v0 prefix="drivewhl_fl"/>
+    <xacro:wheel_gazebo_v0 prefix="drivewhl_fr"/>
+    <xacro:wheel_gazebo_v0 prefix="drivewhl_rl"/>
+    <xacro:wheel_gazebo_v0 prefix="drivewhl_rr"/>
 </robot>

Commit message: Added Lidar camera to simulation

File: src/trr_robot/description/gz.xacro (robot description, xacro)
@@ -57,4 +57,34 @@
         </sensor>
     </gazebo>
+    <!-- ........................... Lidar CAMERA config ................................... -->
+    <gazebo reference="lidar">
+        <sensor name='gpu_lidar' type='gpu_lidar'>
+            <topic>scan</topic>
+            <update_rate>30</update_rate>
+            <gz_frame_id>lidar</gz_frame_id>
+            <lidar>
+                <scan>
+                    <horizontal>
+                        <samples>361</samples>
+                        <resolution>1</resolution>
+                        <min_angle>${radians(0)}</min_angle>
+                        <max_angle>${radians(360)}</max_angle>
+                    </horizontal>
+                </scan>
+                <range>
+                    <min>0.55</min>
+                    <max>16</max>
+                    <resolution>0.01</resolution>
+                </range>
+                <noise>
+                    <type>gaussian</type>
+                    <mean>0.0</mean>
+                    <stddev>0.001</stddev>
+                </noise>
+            </lidar>
+            <always_on>1</always_on>
+            <visualize>true</visualize>
+        </sensor>
+    </gazebo>
     <!-- ........................... Wheels and Base and Stuff ................................... -->
     <xacro:macro name="base_gazebo_v0">

File: src/trr_robot/description/trr_robot.xacro (robot description, xacro)
@@ -74,5 +74,5 @@
     <xacro:wheel prefix="drivewhl_rl" x_reflect="-1" y_reflect="1" />
     <xacro:wheel prefix="drivewhl_rr" x_reflect="-1" y_reflect="-1" />
-    <!-- Depth CAMERA -->
+    <!-- ............................ Depth Camera................................... -->
     <link name="depth_camera">
         <visual>
@@ -80,6 +80,6 @@
                 <box size="0.010 0.03 0.03"/>
             </geometry>
-            <material name="Cyan">
-                <color rgba="0 1.0 1.0 1.0"/>
+            <material name="Green">
+                <color rgba="0.0 1.0 0.0 1.0"/>
             </material>
         </visual>
@@ -96,3 +96,26 @@
         <child link="depth_camera_optical"/>
     </joint>
+    <!-- ............................ LIDAR ................................... -->
+    <link name="lidar">
+        <collision>
+            <origin xyz="0 0 0" rpy="0 0 0" />
+            <geometry>
+                <cylinder length="0.06" radius="0.075"/>
+            </geometry>
+        </collision>
+        <visual>
+            <origin xyz="0 0 0" rpy="0 0 0" />
+            <geometry>
+                <cylinder length="0.06" radius="0.075"/>
+            </geometry>
+            <material name="Red">
+                <color rgba="1.0 0.0 0.0 1.0"/>
+            </material>
+        </visual>
+    </link>
+    <joint name="lidar_joint" type="fixed">
+        <parent link="base_link"/>
+        <child link="lidar"/>
+        <origin xyz="0.0 0 0.08" rpy="0 0 0" />
+    </joint>
 </robot>
