Commit message: Updated controller code

File: src/trr_robot/description/robot.urdf.xacro (robot description, xacro)
@@ -7,7 +7,7 @@
         <xacro:include filename="ros2_control.xacro" />
     </xacro:if>
-    <xacro:unless value="$(arg use_ros2_control)">
+    <!-- <xacro:unless value="$(arg use_ros2_control)">
         <xacro:include filename="gz.xacro" />
-    </xacro:unless>
+    </xacro:unless> -->
     <!-- <xacro:include filename="lidar.xacro" />
     <xacro:include filename="camera.xacro" /> -->

File: src/trr_robot/description/ros2_control.xacro (robot description, xacro)
@@ -1,18 +1,26 @@
 <?xml version="1.0"?>
-<robot>
+<robot xmlns:xacro="http://www.ros.org/wiki/xacro">
     <ros2_control name="ToolRetrievalRobot" type="system">
         <hardware>
-            <plugin>/dependencies/diffdrive_arduino/DiffDriveArduino</plugin>
-            <param name="top_left_name">left_wheel_joint</param>
-            <param name="bottom_left_name">left_wheel_joint</param>
-            <param name="top_right_name">right_wheel_joint</param>
-            <param name="bottom_right_name">right_wheel_joint</param>
+            <plugin>diffdrive_arduino/DiffDriveArduinoHardware</plugin>
+            <param name="left_wheel_name">drivewhl_fl_wheel</param>
+            <param name="right_wheel_name">drivewhl_fr_wheel</param>
+            <!-- <param name="top_right_name">right_wheel_joint</param> -->
+            <!-- <param name="bottom_right_name">right_wheel_joint</param> -->
             <param name="loop_rate">30</param>
             <param name="device">/dev/ttyUSB0</param>
-            <param name="baud_rate">9600</param>
-            <param name="timeout">1000</param>
+            <param name="baud_rate">57600</param>
+            <param name="timeout_ms">1000</param>
             <param name="enc_counts_per_rev">3436</param>
         </hardware>
-        <joint name="top_left_joint">
+        <joint name="drivewhl_fl_wheel">
+            <command_interface name="velocity">
+                <param name="min">-10</param>
+                <param name="max">10</param>
+            </command_interface>
+            <state_interface name="position"/>
+            <state_interface name="velocity"/>
+        </joint>
+        <!-- <joint name="bottom_left_joint">
             <command_interface name="velocity">
                 <param name="min">-10</param>
@@ -21,6 +29,14 @@
             <state_interface name="velocity"/>
             <state_interface name="position"/>
+        </joint> -->
+        <joint name="drivewhl_fr_wheel">
+            <command_interface name="velocity">
+                <param name="min">-10</param>
+                <param name="max">10</param>
+            </command_interface>
+            <state_interface name="position"/>
+            <state_interface name="velocity"/>
         </joint>
-        <joint name="bottom_left_joint">
+        <!-- <joint name="bottom_right_joint">
             <command_interface name="velocity">
                 <param name="min">-10</param>
@@ -29,21 +45,5 @@
             <state_interface name="velocity"/>
             <state_interface name="position"/>
-        </joint>
-        <joint name="top_right_joint">
-            <command_interface name="velocity">
-                <param name="min">-10</param>
-                <param name="max">10</param>
-            </command_interface>
-            <state_interface name="velocity"/>
-            <state_interface name="position"/>
-        </joint>
-        <joint name="bottom_right_joint">
-            <command_interface name="velocity">
-                <param name="min">-10</param>
-                <param name="max">10</param>
-            </command_interface>
-            <state_interface name="velocity"/>
-            <state_interface name="position"/>
-        </joint>
+        </joint> -->
     </ros2_control>
 </robot>

Commit message: Updated arduino script for PID control and ros2 conrol file with all 4 motors

File: src/trr_robot/description/robot.urdf.xacro (robot description, xacro)
@@ -7,7 +7,7 @@
         <xacro:include filename="ros2_control.xacro" />
     </xacro:if>
-    <!-- <xacro:unless value="$(arg use_ros2_control)">
+    <xacro:unless value="$(arg use_ros2_control)">
         <xacro:include filename="gz.xacro" />
-    </xacro:unless> -->
+    </xacro:unless>
     <!-- <xacro:include filename="lidar.xacro" />
     <xacro:include filename="camera.xacro" /> -->

File: src/trr_robot/description/ros2_control.xacro (robot description, xacro)
@@ -12,6 +12,7 @@
             <param name="baud_rate">57600</param>
             <param name="timeout_ms">1000</param>
-            <param name="enc_counts_per_rev">3436</param>
+            <param name="enc_counts_per_rev">64</param>
         </hardware>
+         <!-- Front wheels -->
         <joint name="drivewhl_fl_wheel">
             <command_interface name="velocity">
@@ -22,12 +23,4 @@
             <state_interface name="velocity"/>
         </joint>
-        <!-- <joint name="bottom_left_joint">
-            <command_interface name="velocity">
-                <param name="min">-10</param>
-                <param name="max">10</param>
-            </command_interface>
-            <state_interface name="velocity"/>
-            <state_interface name="position"/>
-        </joint> -->
         <joint name="drivewhl_fr_wheel">
             <command_interface name="velocity">
@@ -38,11 +31,20 @@
             <state_interface name="velocity"/>
         </joint>
-        <!-- <joint name="bottom_right_joint">
+         <!-- Back wheels -->
+         <!-- <joint name="drivewhl_bl_wheel">
             <command_interface name="velocity">
                 <param name="min">-10</param>
                 <param name="max">10</param>
             </command_interface>
+            <state_interface name="position"/>
             <state_interface name="velocity"/>
+        </joint>
+        <joint name="drivewhl_br_wheel">
+            <command_interface name="velocity">
+                <param name="min">-10</param>
+                <param name="max">10</param>
+            </command_interface>
             <state_interface name="position"/>
+            <state_interface name="velocity"/>
         </joint> -->
     </ros2_control>
