Commit message: Attaching basic camera to simulated robot

File: src/trr_robot/description/ros2_control.xacro (robot description, xacro)
@@ -43,4 +43,9 @@
       </joint>
     </ros2_control>
+    <gazebo>
+      <plugin filename="gz_ros2_control-system" name="gz_ros2_control::GazeboSimROS2ControlPlugin">
+        <parameters>$(find trr_robot_desc)/config/trr_robot_sim.yaml</parameters>
+      </plugin>
+    </gazebo>
   </xacro:macro>
 </robot>

File: src/trr_robot/description/trr_robot.urdf.xacro (robot description, xacro)
@@ -1,99 +1,5 @@
 <?xml version="1.0"?>
-<!-- ros2 launch trr_controller display.launch.py -->
 <robot xmlns:xacro="http://www.ros.org/wiki/xacro" name="trr_robot">
-    <xacro:include filename="$(find trr_robot_desc)/gazebo/trr_robot.gazebo.xacro" />
-    <xacro:include filename="$(find trr_robot_desc)/ros2_control/trr_robot.ros2_control.xacro" />
-    <xacro:property name="base_width" value="0.4572"/>
-    <xacro:property name="base_length" value="0.5588"/>
-    <xacro:property name="base_height" value="0.0762"/>
-    <xacro:property name="wheel_radius" value="0.05"/>
-    <xacro:property name="wheel_width" value="0.04"/>
-    <xacro:property name="wheel_ygap" value="0.0127"/>
-    <xacro:property name="wheel_zoff" value="0.0381"/>
-    <xacro:property name="wheel_xoff" value="0.215"/>
-    <!-- =============== Link & Joint =============== -->
-    <link name="base_footprint"></link>
-    <joint name="base_joint" type="fixed">
-        <parent link="base_footprint"/>
-        <child link="base_link"/>
-        <origin xyz="0.0 0.0 0.075" rpy="0 0 0"/>
-    </joint>
-    <link name="base_link">
-        <visual>
-            <geometry>
-                <box size="${base_length} ${base_width} ${base_height}"/>
-            </geometry>
-            <material name="Cyan">
-                <color rgba="0 1.0 1.0 1.0"/>
-            </material>
-        </visual>
-        <collision>
-            <origin xyz="0 0 0.05" rpy="0 0 0"/>
-            <geometry>
-                <box size="${base_length} ${base_width} ${base_height}"/>
-            </geometry>
-        </collision>
-        <inertial>
-            <origin xyz="0 0 0.05" rpy="0 0 0"/>
-            <mass value="12"/>
-            <inertia ixx="2.26" ixy="0.0" ixz="0.0" iyy="6.26" iyz="0.0" izz="8.5"/>
-        </inertial>
-    </link>
-    <!-- Wheels -->
-    <xacro:macro name="wheel" params="prefix x_reflect y_reflect">
-        <link name="${prefix}_link">
-            <visual>
-                <origin xyz="0 0 0" rpy="${pi/2} 0 0"/>
-                <geometry>
-                    <cylinder radius="${wheel_radius}" length="${wheel_width}"/>
-                </geometry>
-                <material name="Gray">
-                <color rgba="0.5 0.5 0.5 1.0"/>
-                </material>
-            </visual>
-            <collision>
-                <origin xyz="0 0 0" rpy="${pi/2} 0 0"/>
-                <geometry>
-                    <cylinder radius="${wheel_radius}" length="${wheel_width}"/>
-                </geometry>
-            </collision>
-            <inertial>
-                <origin xyz="0 0 0"/>
-                <mass value="0.05"/>
-                <inertia ixx="0.00001" ixy="0" ixz="0" iyy="0.000018" iyz="0" izz="0.00001"/>
-            </inertial>
-        </link>
-        <joint name="${prefix}_joint" type="continuous">
-            <parent link="base_link"/>
-            <child link="${prefix}_link"/>
-            <origin xyz="${x_reflect*wheel_xoff} ${y_reflect*(base_width/2+wheel_ygap)} ${-wheel_zoff}" rpy="0 0 0"/>
-            <axis xyz="0 1 0"/>
-        </joint>
-    </xacro:macro>
-    <xacro:wheel prefix="drivewhl_fl" x_reflect="1" y_reflect="1" />
-    <xacro:wheel prefix="drivewhl_fr" x_reflect="1" y_reflect="-1" />
-    <xacro:wheel prefix="drivewhl_rl" x_reflect="-1" y_reflect="1" />
-    <xacro:wheel prefix="drivewhl_rr" x_reflect="-1" y_reflect="-1" />
-    <!-- =============== Gazebo =============== -->
-    <xacro:macro name="base_gazebo_v0">
-        <gazebo reference="base_link">
-            <selfCollide>false</selfCollide>
-            <mu1 value="0.05" />
-            <mu2 value="0.05" />
-        </gazebo>
-    </xacro:macro>
-    <xacro:macro name="wheel_gazebo_v0" params="prefix">
-        <gazebo reference="${prefix}_link">
-            <selfCollide>false</selfCollide>
-            <mu1 value="1.2" />
-            <mu2 value="1.2" />
-        </gazebo>
-    </xacro:macro>
-    <xacro:base_gazebo_v0/>
-    <xacro:wheel_gazebo_v0 prefix="drivewhl_fl"/>
-    <xacro:wheel_gazebo_v0 prefix="drivewhl_fr"/>
-    <xacro:wheel_gazebo_v0 prefix="drivewhl_rl"/>
-    <xacro:wheel_gazebo_v0 prefix="drivewhl_rr"/>
-    <xacro:trr_robot_gazebo/>
-    <xacro:trr_robot_ros2_control/>
+    <xacro:include filename="robot_core.xacro"/>
+    <xacro:include filename="depth_camera.xacro" />
 </robot>

Commit message: Working changes

File: src/trr_robot/description/ros2_control.xacro (robot description, xacro)
@@ -6,11 +6,9 @@
             <param name="left_wheel_name">drivewhl_fl_wheel</param>
             <param name="right_wheel_name">drivewhl_fr_wheel</param>
-            <!-- <param name="top_right_name">right_wheel_joint</param> -->
-            <!-- <param name="bottom_right_name">right_wheel_joint</param> -->
             <param name="loop_rate">30</param>
             <param name="device">/dev/ttyUSB0</param>
             <param name="baud_rate">57600</param>
             <param name="timeout_ms">1000</param>
-            <param name="enc_counts_per_rev">64</param>
+            <param name="enc_counts_per_rev">550</param>
         </hardware>
          <!-- Front wheels -->

File: src/trr_robot/description/trr_robot.xacro (robot description, xacro)
@@ -4,5 +4,5 @@
     <xacro:property name="base_length" value="0.5588"/>
     <xacro:property name="base_height" value="0.0762"/>
-    <xacro:property name="wheel_radius" value="0.05"/>
+    <xacro:property name="wheel_radius" value="0.04"/>
     <xacro:property name="wheel_width" value="0.04"/>
     <xacro:property name="wheel_ygap" value="0.0127"/>
