Commit message: Adding mapping rviz visualizer and fixing laser transform frame

File: perceptron_ws/src/generic/trr_bringup/description/trr_robot.xacro (robot description, xacro)
@@ -95,5 +95,5 @@
     </joint>
     <!-- ............................ LIDAR ................................... -->
-    <link name="lidar">
+    <link name="laser">
         <collision>
             <origin xyz="0 0 0" rpy="0 0 0" />
@@ -112,7 +112,7 @@
         </visual>
     </link>
-    <joint name="lidar_joint" type="fixed">
+    <joint name="laser_joint" type="fixed">
         <parent link="base_link"/>
-        <child link="lidar"/>
+        <child link="laser"/>
         <origin xyz="0.0 0 0.08" rpy="0 0 0" />
     </joint>
